File: sanjogknowspcb.kicad_pcb (KiCad board)
At the start: 2 copper layers, 66.4 x 36.7 mm, 13 parts, among them SW1 SW_Push

Commit message: Add files via upload
Parts:
- added G***: LOGO, LOGO, B.Cu at (131.5, 122.8)
- added G***: LOGO, LOGO, B.Cu at (91.2, 124.5)

Commit message: Add files via upload
Parts:
- added Q1: NPN, Package_TO_SOT_THT:TO-92L_HandSolder, F.Cu at (90.0, 124.0)
- added R8: R, Resistor_THT:R_Axial_DIN0207_L6.3mm_D2.5mm_P7.62mm_Horizontal, F.Cu at (89.5, 117.8)
Connections:
- D1 pad 1: Net-(BT1--) -> Net-(D1-K)
- D2 pad 1: Net-(BT1--) -> Net-(D1-K)
- D3 pad 1: Net-(BT1--) -> Net-(D1-K)
- SW1 pad 2: Net-(R1-Pad1) -> Net-(R1-Pad2)
Routing:
- net Net-(D1-K): track 0.00 -> 59.8 mm
- net Net-(BT1--): track 78.6 -> 24.1 mm
- net Net-(R1-Pad1): track 22.4 -> 52.9 mm
- net Net-(D3-A): track 37.4 -> 17.2 mm
- net Net-(R1-Pad2): track 80.2 -> 92.8 mm
- net Net-(BT1-+): track 85.1 -> 78.3 mm
- net Net-(Q1-B): track 0.00 -> 5.70 mm
